File: hw/powerboard/powerboard.sch (EAGLE design)
At the start: 37 parts, among them J1 ISP, J2 I2C

Commit message: Recent progress with powerboard schematics
Parts:
- added BATTERY: (no value), con-wago-500:W237-102
- added Q1: IRF4905, transistor-power:IRF4905
- D1: value BAT -> BATT
Connections:
- net V_BATT_ADC renamed 12V_ADC
- removed net V_BATT: C6.1, D1.A, F1.2, J3.1, L1.1, R1.2
- new net 12V: C6.1, D1.A, J3.1, L1.1, Q1.S, R1.2
- new net N$11: BATTERY-1.KL, F1.2
- new net N$9: F1.1, Q1.D
- net GND: now also BATTERY-2.KL, Q1.G
Changed lines of the file:
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@@
 <part name="GND2" library="SparkFun-Aesthetics" deviceset="GND" device=""/>
 <part name="C1" library="SparkFun-Capacitors" deviceset="CAP" device="0603-CAP"/>
-<part name="SUPPLY2" library="SparkFun-Aesthetics" deviceset="V_BATT" device=""/>
 <part name="R4" library="SparkFun-Passives" deviceset="RESISTOR" device="0603-RES"/>
 <part name="R5" library="SparkFun-Passives" deviceset="RESISTOR" device="0603-RES"/>
@@
 <part name="C5" library="SparkFun-Capacitors" deviceset="CAP" device="0603-CAP" value="100nF"/>
 <part name="F1" library="SparkFun-Passives" deviceset="FUSE" device="X20MM"/>
-<part name="SUPPLY6" library="SparkFun-Aesthetics" deviceset="V_BATT" device=""/>
-<part name="GND6" library="SparkFun-Aesthetics" deviceset="GND" device=""/>
 <part name="SUPPLY4" library="SparkFun-Aesthetics" deviceset="5V" device=""/>
 <part name="SUPPLY3" library="SparkFun-Aesthetics" deviceset="1.8V" device=""/>
@@
 <part name="J2" library="pinhead" deviceset="PINHD-1X3" device="/90" value="I2C"/>
 <part name="GND8" library="SparkFun-Aesthetics" deviceset="GND" device=""/>
-<part name="D1" library="SparkFun-LED" deviceset="LED" device="0603" value="BAT"/>
+<part name="D1" library="SparkFun-LED" deviceset="LED" device="0603" value="BATT"/>
 <part name="D2" library="SparkFun-LED" deviceset="LED" device="0603" value="5V"/>
 <part name="D3" library="SparkFun-LED" deviceset="LED" device="0603" value="3.3V"/>
@@
 <part name="R15" library="SparkFun-Passives" deviceset="RESISTOR" device="0603-RES"/>
 <part name="R16" library="SparkFun-Passives" deviceset="RESISTOR" device="0603-RES"/>
-<part name="SUPPLY8" library="SparkFun-Aesthetics" deviceset="V_BATT" device=""/>
 <part name="SUPPLY9" library="SparkFun-Aesthetics" deviceset="5V" device=""/>
 <part name="SUPPLY10" library="SparkFun-Aesthetics" deviceset="3.3V" device=""/>
@@
 <part name="L1" library="WE-HCI" deviceset="WE-HCI" device="_7030/7040/7050" technology="-744314650"/>
 <part name="GND14" library="SparkFun-Aesthetics" deviceset="GND" device=""/>
-<part name="SUPPLY13" library="SparkFun-Aesthetics" deviceset="V_BATT" device=""/>
 <part name="U$2" library="powerboard" deviceset="AXA04AXX-L" device=""/>
+<part name="SUPPLY14" library="SparkFun-Aesthetics" deviceset="12V" device=""/>
+<part name="SUPPLY8" library="SparkFun-Aesthetics" deviceset="12V" device=""/>
+<part name="SUPPLY13" library="SparkFun-Aesthetics" deviceset="12V" device=""/>
+<part name="SUPPLY2" library="SparkFun-Aesthetics" deviceset="12V" device=""/>
+<part name="Q1" library="transistor-power" deviceset="IRF4905" device=""/>
+<part name="GND6" library="SparkFun-Aesthetics" deviceset="GND" device=""/>
+<part name="BATTERY" library="con-wago-500" deviceset="W237-102" device=""/>
 </parts>
 <sheets>
@@
 <instance part="GND2" gate="1" x="27.94" y="124.46"/>
 <instance part="C1" gate="G$1" x="48.26" y="134.62"/>
-<instance part="SUPPLY2" gate="G$1" x="27.94" y="160.02"/>
 <instance part="R4" gate="G$1" x="27.94" y="78.74" rot="R90"/>
 <instance part="R5" gate="G$1" x="27.94" y="63.5" rot="R90"/>
@@
 <instance part="C5" gate="G$1" x="154.94" y="144.78"/>
 <instance part="F1" gate="G$1" x="58.42" y="246.38" rot="R180"/>
-<instance part="SUPPLY6" gate="G$1" x="40.64" y="246.38" rot="R90"/>
-<instance part="GND6" gate="1" x="38.1" y="223.52" rot="R270"/>
 <instance part="SUPPLY4" gate="G$1" x="27.94" y="86.36"/>
 <instance part="SUPPLY3" gate="G$1" x="93.98" y="86.36"/>
@@
 <instance part="R15" gate="G$1" x="124.46" y="175.26" rot="R180"/>
 <instance part="R16" gate="G$1" x="124.46" y="101.6" rot="R180"/>
-<instance part="SUPPLY8" gate="G$1" x="27.94" y="175.26" rot="R90"/>
 <instance part="SUPPLY9" gate="G$1" x="27.94" y="101.6" rot="R90"/>
 <instance part="SUPPLY10" gate="G$1" x="93.98" y="175.26" rot="R90"/>
@@
 <instance part="L1" gate="G$1" x="157.48" y="233.68"/>
 <instance part="GND14" gate="1" x="149.86" y="215.9"/>
-<instance part="SUPPLY13" gate="G$1" x="147.32" y="233.68" rot="R90"/>
 <instance part="U$2" gate="G$1" x="172.72" y="238.76"/>
+<instance part="SUPPLY14" gate="G$1" x="96.52" y="246.38" rot="R270"/>
+<instance part="SUPPLY8" gate="G$1" x="147.32" y="233.68" rot="R90"/>
+<instance part="SUPPLY13" gate="G$1" x="27.94" y="175.26" rot="R90"/>
+<instance part="SUPPLY2" gate="G$1" x="27.94" y="160.02"/>
+<instance part="Q1" gate="G$1" x="76.2" y="243.84" rot="MR90"/>
+<instance part="GND6" gate="1" x="73.66" y="231.14"/>
+<instance part="BATTERY" gate="-1" x="38.1" y="246.38"/>
+<instance part="BATTERY" gate="-2" x="38.1" y="236.22"/>
 </instances>
 <busses>
@@
 <pinref part="U$2" gate="G$1" pin="-VIN"/>
 </segment>
+<segment>
+<pinref part="Q1" gate="G$1" pin="G"/>
+<pinref part="GND6" gate="1" pin="GND"/>
+<wire x1="73.66" y1="238.76" x2="73.66" y2="236.22" width="0.1524" layer="91"/>
+<pinref part="BATTERY" gate="-2" pin="KL"/>
+<wire x1="73.66" y1="236.22" x2="73.66" y2="233.68" width="0.1524" layer="91"/>
+<wire x1="43.18" y1="236.22" x2="73.66" y2="236.22" width="0.1524" layer="91"/>
+<junction x="73.66" y="236.22"/>
+</segment>
 </net>
 <net name="N$1" class="0">
@@
 <wire x1="27.94" y1="144.78" x2="27.94" y2="142.24" width="0.1524" layer="91"/>
 <wire x1="27.94" y1="144.78" x2="33.02" y2="144.78" width="0.1524" layer="91"/>
-</segment>
-</net>
-<net name="V_BATT_ADC" class="0">
-<segment>
-<pinref part="R3" gate="G$1" pin="1"/>
-<pinref part="C1" gate="G$1" pin="1"/>
-<wire x1="43.18" y1="144.78" x2="48.26" y2="144.78" width="0.1524" layer="91"/>
-<wire x1="48.26" y1="144.78" x2="48.26" y2="139.7" width="0.1524" layer="91"/>
-<wire x1="48.26" y1="144.78" x2="66.04" y2="144.78" width="0.1524" layer="91"/>
-<junction x="66.04" y="144.78"/>
-<label x="50.8" y="144.78" size="1.778" layer="95"/>
-</segment>
-<segment>
-<pinref part="U$1" gate="G$1" pin="(PCINT0/AREF/ADC0)PA0"/>
-<wire x1="210.82" y1="129.54" x2="231.14" y2="129.54" width="0.1524" layer="91"/>
-<junction x="231.14" y="129.54"/>
-<label x="213.36" y="129.54" size="1.778" layer="95"/>
-</segment>
-</net>
-<net name="V_BATT" class="0">
-<segment>
-<pinref part="R1" gate="G$1" pin="2"/>
-<wire x1="27.94" y1="157.48" x2="27.94" y2="160.02" width="0.1524" layer="91"/>
-<pinref part="SUPPLY2" gate="G$1" pin="V_BATT"/>
-</segment>
-<segment>
-<pinref part="SUPPLY6" gate="G$1" pin="V_BATT"/>
-<pinref part="F1" gate="G$1" pin="2"/>
-<wire x1="40.64" y1="246.38" x2="48.26" y2="246.38" width="0.1524" layer="91"/>
-</segment>
-<segment>
-<pinref part="SUPPLY8" gate="G$1" pin="V_BATT"/>
-<pinref part="D1" gate="G$1" pin="A"/>
-<wire x1="27.94" y1="175.26" x2="35.56" y2="175.26" width="0.1524" layer="91"/>
-<pinref part="J3" gate="G$1" pin="1"/>
-<wire x1="35.56" y1="175.26" x2="43.18" y2="175.26" width="0.1524" layer="91"/>
-<junction x="35.56" y="175.26"/>
-</segment>
-<segment>
-<pinref part="L1" gate="G$1" pin="1"/>
-<pinref part="C6" gate="G$1" pin="1"/>
-<wire x1="152.4" y1="233.68" x2="149.86" y2="233.68" width="0.1524" layer="91"/>
-<wire x1="149.86" y1="233.68" x2="149.86" y2="231.14" width="0.1524" layer="91"/>
-<wire x1="149.86" y1="233.68" x2="147.32" y2="233.68" width="0.1524" layer="91"/>
-<junction x="149.86" y="233.68"/>
-<pinref part="SUPPLY13" gate="G$1" pin="V_BATT"/>
 </segment>
 </net>
@@
 </segment>
 </net>
+<net name="12V" class="0">
+<segment>
+<pinref part="L1" gate="G$1" pin="1"/>
+<pinref part="C6" gate="G$1" pin="1"/>
+<wire x1="152.4" y1="233.68" x2="149.86" y2="233.68" width="0.1524" layer="91"/>
+<wire x1="149.86" y1="233.68" x2="149.86" y2="231.14" width="0.1524" layer="91"/>
+<wire x1="149.86" y1="233.68" x2="147.32" y2="233.68" width="0.1524" layer="91"/>
+<junction x="149.86" y="233.68"/>
+<pinref part="SUPPLY8" gate="G$1" pin="12V"/>
+</segment>
+<segment>
+<pinref part="D1" gate="G$1" pin="A"/>
+<wire x1="27.94" y1="175.26" x2="35.56" y2="175.26" width="0.1524" layer="91"/>
+<pinref part="J3" gate="G$1" pin="1"/>
+<wire x1="35.56" y1="175.26" x2="43.18" y2="175.26" width="0.1524" layer="91"/>
+<junction x="35.56" y="175.26"/>
+<pinref part="SUPPLY13" gate="G$1" pin="12V"/>
+</segment>
+<segment>
+<pinref part="R1" gate="G$1" pin="2"/>
+<wire x1="27.94" y1="157.48" x2="27.94" y2="160.02" width="0.1524" layer="91"/>
+<pinref part="SUPPLY2" gate="G$1" pin="12V"/>
+</segment>
+<segment>
+<pinref part="Q1" gate="G$1" pin="S"/>
+<pinref part="SUPPLY14" gate="G$1" pin="12V"/>
+<wire x1="81.28" y1="246.38" x2="96.52" y2="246.38" width="0.1524" layer="91"/>
+</segment>
+</net>
+<net name="12V_ADC" class="0">
+<segment>
+<pinref part="R3" gate="G$1" pin="1"/>
+<pinref part="C1" gate="G$1" pin="1"/>
+<wire x1="43.18" y1="144.78" x2="48.26" y2="144.78" width="0.1524" layer="91"/>
+<wire x1="48.26" y1="144.78" x2="48.26" y2="139.7" width="0.1524" layer="91"/>
+<wire x1="48.26" y1="144.78" x2="66.04" y2="144.78" width="0.1524" layer="91"/>
+<junction x="66.04" y="144.78"/>
+<label x="50.8" y="144.78" size="1.778" layer="95"/>
+</segment>
+<segment>
+<pinref part="U$1" gate="G$1" pin="(PCINT0/AREF/ADC0)PA0"/>
+<wire x1="210.82" y1="129.54" x2="231.14" y2="129.54" width="0.1524" layer="91"/>
+<junction x="231.14" y="129.54"/>
+<label x="213.36" y="129.54" size="1.778" layer="95"/>
+</segment>
+</net>
+<net name="N$9" class="0">
+<segment>
+<pinref part="F1" gate="G$1" pin="1"/>
+<pinref part="Q1" gate="G$1" pin="D"/>
+<wire x1="68.58" y1="246.38" x2="71.12" y2="246.38" width="0.1524" layer="91"/>
+</segment>
+</net>
+<net name="N$11" class="0">
+<segment>
+<pinref part="BATTERY" gate="-1" pin="KL"/>
+<pinref part="F1" gate="G$1" pin="2"/>
+<wire x1="43.18" y1="246.38" x2="48.26" y2="246.38" width="0.1524" layer="91"/>
+</segment>
+</net>
