File: hw/powersensor/powersensor.brd (EAGLE design)
At the start: 26.3 x 31.1 mm, 37 parts, among them J1 ISP, J2 I2C

Commit message: Removed cruft
Parts:
- removed J9: (no value), SparkFun-Connectors:1X01
- added U$3: (no value), SparkFun-Aesthetics:OSHW-LOGO-M
- J2: device pinhead:1X03/90 -> pinhead:1X04/90
- J8: device SparkFun-Connectors:1X06 -> SparkFun-Connectors:1X05
- U$1: value ATTINY84 -> ATTINYx4
- moved C5 3.82 mm to (5.56, 2.86), turned to 90 degrees
- moved R17 1.28 mm to (8.89, 9.21)
- moved R18 1.28 mm to (8.89, 6.67)
- moved J8 1.27 mm to (18.1, 2.86)
Connections:
- net CURRENT_B renamed CURRENT
- removed net CURRENT_A: J8.3, U$1.10
- removed net MISO/1.8V_ADC: C4.1, J1.1, R12.1, U$1.8
- new net 1.8V_ADC: C4.1, R12.1, U$1.10
- new net MISO: J1.1, U$1.8
- net GND: no longer J9.1
- net PB0: now also J8.4; no longer J8.5
- net PB1: now also J8.3; no longer J8.4
- net VIN: now also J2.4, J8.5; no longer J8.6
Routing:
- net 1.8V_ADC: track 0.00 -> 11.4 mm
- net MISO/1.8V_ADC: track 10.7 -> 0.00 mm
- net CURRENT_A: track 10.4 -> 0.00 mm, vias 1 -> 0
- net VIN: track 31.8 -> 39.7 mm
- net MISO: track 0.00 -> 4.39 mm
- net SDA/MOSI: track 24.4 -> 27.2 mm
- net CURRENT: track 5.72 -> 4.82 mm
- net PB1: track 4.82 -> 5.35 mm
- net PB0: track 5.35 -> 4.82 mm
Other:
- outline, holes or cut-outs redrawn
- board text added: "CURR"
- board text added: "PowerSensor v0.2"
- board text added: "designed by: Hanno Gerd Meyer 12/2016"
- board text added: "v0.2"
- board text removed: "C_A"
- board text removed: "C_B"
- board text removed: "PowerSensor v0.1"
- board text removed: "designed by: Hanno Gerd Meyer November, 2016"
