File: hw/powersensor/powersensor.sch (EAGLE design)
At the start: 37 parts, among them J1 ISP, J2 I2C

Commit message: Removed cruft
Parts:
- removed J9: (no value), SparkFun-Connectors:M01PTH
- J2: device pinhead:PINHD-1X3/90 -> pinhead:PINHD-1X4/90
- J8: device SparkFun-Connectors:M06SILK_FEMALE_PTH -> SparkFun-Connectors:M05PTH
- U$1: value ATTINY84 -> ATTINYx4
Connections:
- net CURRENT_B renamed CURRENT
- removed net CURRENT_A: J8.3, U$1.(PCINT3/T0/ADC3)PA3
- removed net MISO/1.8V_ADC: C4.1, J1.1, R12.1, U$1.(PCINT5/OC1B/MISO/DO/ADC5)PA5
- new net 1.8V_ADC: C4.1, R12.1, U$1.(PCINT3/T0/ADC3)PA3
- new net MISO: J1.1, U$1.(PCINT5/OC1B/MISO/DO/ADC5)PA5
- net GND: no longer J9.1
- net PB0: now also J8.4; no longer J8.5
- net PB1: now also J8.3; no longer J8.4
- net VIN: now also J2.4, J8.5; no longer J8.6
Other:
- moved on the sheet: J7
